File: clk_led_matrix.kicad_sch (KiCad schematic)
At the start: 58 parts, among them J1 USB_C_Receptacle_USB2.0_16P, J10 LED_MATRIX_0, J2 LED_MATRIX_0, J3 CH32_prog, J4 STM32_prog, J5 Conn_Coaxial, J6 LED_MATRIX_0, J7 LED_MATRIX_0, J8 LED_MATRIX_0, J9 LED_MATRIX_0, SW1 RST, SW2 BOOT, U1 STM32C071KBUx, U2 AMS1117-3.3, U3 ATGM336H-5N31, Y1 Q13FC13500004

Commit message: update layout and usb c connector
Parts:
- removed R3: 0, Resistor_SMD:R_0603_1608Metric, symbol Device:R
- added H1, H2, H3, H4: MountingHole_Pad, MountingHole:MountingHole_3.2mm_M3_Pad_Via, symbol Mechanical:MountingHole_Pad
- J1: footprint Connector_USB:USB_C_Receptacle_GCT_USB4115-03-C -> easyeda2kicad:USB-C-TH_SHOUHAN_TYPE-C-14PLC-H10.0
Connections:
- net GND: now also J1.SH (SHIELD), H1.1, H2.1, H3.1, H4.1

Commit message: update schematic and layout
Parts:
- added Q1: 2N7002, Package_TO_SOT_SMD:SOT-23, symbol Transistor_FET:2N7002
- added R24: 5k1, Resistor_SMD:R_0603_1608Metric, symbol Device:R
- added TP3: RTC_OUT, TestPoint:TestPoint_Pad_D1.0mm, symbol Connector:TestPoint
- added TP4: GNSS, TestPoint:TestPoint_Pad_D1.0mm, symbol Connector:TestPoint
- R20, R21, R22, R23: value 5k1 -> 100
- SW1, SW2: LCSC (none) -> C720477
- U3: LCSC (none) -> C90770; LCSC Part C90770 -> (none)
- Y1: LCSC (none) -> C32346
Connections:
- net GND: now also Q1.2 (S), R24.1; no longer D4.1 (K), D5.1 (K), D6.1 (K), D7.1 (K)
- net GNSS_I2C_SCL: now also TP3.1
- net GNSS_I2C_SDA: now also TP4.1
- net LED_DRIVE: now reaches U1.27 (PB3)
- net LED_DRIVE: now also Q1.1 (G), R24.2
- new net: D4.1 (K), D5.1 (K), D6.1 (K), D7.1 (K), Q1.3 (D)
